File: Hardware/Qwiic_1.8V_Adapter.brd (EAGLE design)
At the start: 25.4 x 25.4 mm, 47 parts, among them J1 QWIIC_RIGHT_ANGLE, J2 QWIIC_RIGHT_ANGLE, U3 AP2127K-1.8V

Commit message: Add EN Jumper note
Parts:
- renumbered JP1 to EN
Changed lines of the file:
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@@
 <layer number="44" name="Drills" color="7" fill="1" visible="no" active="yes"/>
 <layer number="45" name="Holes" color="7" fill="1" visible="yes" active="yes"/>
-<layer number="46" name="Milling" color="3" fill="1" visible="yes" active="yes"/>
+<layer number="46" name="Milling" color="3" fill="1" visible="no" active="yes"/>
 <layer number="47" name="Measures" color="7" fill="1" visible="no" active="yes"/>
 <layer number="48" name="Document" color="7" fill="1" visible="no" active="yes"/>
@@
 <attribute name="VALUE" x="7.62" y="-0.762" size="0.6096" layer="27" font="vector" ratio="20"/>
 </element>
-<element name="JP1" library="SparkFun-Jumpers" package="SMT-JUMPER_3_1-NC_TRACE_SILK" package3d_urn="urn:adsk.eagle:package:39288/1" value="JUMPER-SMT_3_1-NC_TRACE_SILK" x="16.51" y="17.78" smashed="yes" rot="MR0">
+<element name="EN" library="SparkFun-Jumpers" package="SMT-JUMPER_3_1-NC_TRACE_SILK" package3d_urn="urn:adsk.eagle:package:39288/1" value="JUMPER-SMT_3_1-NC_TRACE_SILK" x="16.51" y="17.78" smashed="yes" rot="MR0">
 <attribute name="NAME" x="16.51" y="18.923" size="0.6096" layer="26" font="vector" ratio="20" rot="MR0" align="bottom-center"/>
 <attribute name="VALUE" x="16.51" y="16.637" size="0.6096" layer="28" font="vector" ratio="20" rot="MR0" align="top-center"/>
@@
 <contactref element="R11" pad="1"/>
 <contactref element="C6" pad="2"/>
-<contactref element="JP1" pad="3"/>
+<contactref element="EN" pad="3"/>
 <wire x1="16.09" y1="13.97" x2="16.427" y2="14.307" width="0.2032" layer="1"/>
 <wire x1="16.427" y1="14.307" x2="16.51" y2="14.39" width="0.2032" layer="1"/>
@@
 <signal name="N$1">
 <contactref element="U4" pad="P8"/>
-<contactref element="JP1" pad="2"/>
+<contactref element="EN" pad="2"/>
 <wire x1="18.441" y1="18.389" x2="17.78" y2="19.05" width="0.2032" layer="1"/>
 <wire x1="17.78" y1="19.05" x2="16.51" y2="19.05" width="0.2032" layer="1"/>
@@
 </signal>
 <signal name="EN">
-<contactref element="JP1" pad="1"/>
+<contactref element="EN" pad="1"/>
 <contactref element="J4" pad="5"/>
 <wire x1="17.5514" y1="17.78" x2="17.78" y2="18.0086" width="0.2032" layer="16"/>

Commit message: Production Files and README
Parts:
- added JP1: JUMPER-SMT_2_NC_TRACE_SILK, SparkFun-Jumpers:SMT-JUMPER_2_NC_TRACE_SILK
- added U$30: (no value), output:#LED#0
- moved R5 0.25 mm to (13.0, 10.2)
- moved R10 0.25 mm to (9.14, 10.2)
- moved C6 0.13 mm to (16.4, 15.2)
- moved D1 0.13 mm to (2.54, 6.86)
- moved C4 0.13 mm to (7.75, 15.2)
- moved C5 0.13 mm to (12.6, 15.2)
- moved R11 0.13 mm to (14.1, 15.2)
Connections:
- new net N$3: JP1.1, R1.1
- net 3.3V: now also JP1.2; no longer R1.1
Routing:
- net N$3: track 0.00 -> 14.9 mm, vias 0 -> 1
- net 3.3V: track 59.6 -> 59.3 mm, vias 4 -> 5
- net GND: vias 54 -> 51
